File: ILV2-7-5_Clock/ILV2-7-5_Clock.sch (KiCad schematic (older format))
At the start: 61 parts, among them J1 CONN_01X05, J2 USB_OTG, Q1 BSS84, Q2 BSS138, Q3 BSS84, Q4 BSS138, SW1 TACT_SWITCH, SW2 TACT_SWITCH, SW3 CJS1200, U1 DS3231M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

Commit message: Small update
Parts:
- gave numbers to parts that had none: 1
Changed lines of the file:
@@
 Connection ~ 7700 3000
 $Comp
-L TACT_SWITCH SW?
+L TACT_SWITCH SW4
 U 1 1 5A08B7A0
 P 5150 2800
-F 0 "SW?" H 5150 2750 50  0000 C CNN
+F 0 "SW4" H 5150 2750 50  0000 C CNN
 F 1 "TACT_SWITCH" H 5150 2950 50  0000 C CNN
 F 2 "OpenBCI:PTS810" H 5150 2800 50  0001 C CNN

Commit message: More progress on the PCB and casing down schem issues
Parts:
- added C21: 1uF, Capacitors_SMD:C_0603, symbol C
- SW3: value CJS1200 -> PCM12SMTR; footprint OpenBCI:CJS-1200TA -> Solutions:PCM12SMTR
Connections:
- net labels removed: BATT_LEVEL
- wire segments 191 -> 194
