File: ILV2-7-5_Clock/ILV2-7-5_Clock.sch (KiCad schematic (older format))
At the start: 62 parts, among them J1 CONN_01X05, J2 USB_OTG, Q1 BSS84, Q2 BSS138, Q3 BSS84, Q4 BSS138, SW1 TACT_SWITCH, SW2 TACT_SWITCH, SW3 PCM12SMTR, SW4 TACT_SWITCH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

Commit message: Some more such
Parts:
- J1: footprint Pin_Headers:Pin_Header_Straight_1x05_Pitch1.00mm -> Pin_Headers:Pin_Header_Straight_1x05_Pitch2.54mm
- L1: footprint Capacitors_SMD:C_0603 -> Capacitors_SMD:C_1210
Other:
- note added: "18\n0\n1\n2\n3\n4\n5\n6/A0\n7/A1\n8/A2\n"
- note added: "9/A3\n10/A4\n11/A5\n12/A6\n13/A7\n14/A8\n15\n16\n17"
Changed lines of the file:
@@
 F 0 "J1" H 5500 1700 50  0000 C CNN
 F 1 "CONN_01X05" V 5600 1400 50  0000 C CNN
-F 2 "Pin_Headers:Pin_Header_Straight_1x05_Pitch1.00mm" H 5500 1400 50  0001 C CNN
+F 2 "Pin_Headers:Pin_Header_Straight_1x05_Pitch2.54mm" H 5500 1400 50  0001 C CNN
 F 3 "" H 5500 1400 50  0001 C CNN
 	1    5500 1400
@@
 F 0 "L1" V 11000 2750 50  0000 C CNN
 F 1 "10uH 1.2A" V 11125 2750 50  0000 C CNN
-F 2 "Capacitors_SMD:C_0603" H 11050 2750 50  0001 C CNN
+F 2 "Capacitors_SMD:C_1210" H 11050 2750 50  0001 C CNN
 F 3 "" H 11050 2750 50  0001 C CNN
 	1    11050 2750
@@
 INT/SQW
 $Comp
-L +5V #PWR029
+L +5V #PWR028
 U 1 1 5A1216E5
 P 8500 900
-F 0 "#PWR029" H 8500 750 50  0001 C CNN
+F 0 "#PWR028" H 8500 750 50  0001 C CNN
 F 1 "+5V" H 8500 1040 50  0000 C CNN
 F 2 "" H 8500 900 50  0001 C CNN
@@
 Connection ~ 11000 1050
 $Comp
-L +5V #PWR031
+L +5V #PWR029
 U 1 1 5A122390
 P 6900 1850
-F 0 "#PWR031" H 6900 1700 50  0001 C CNN
+F 0 "#PWR029" H 6900 1700 50  0001 C CNN
 F 1 "+5V" H 6900 1990 50  0000 C CNN
 F 2 "" H 6900 1850 50  0001 C CNN
@@
 	9500 1050 9400 1050
 $Comp
-L +3V3 #PWR032
+L +3V3 #PWR030
 U 1 1 5A123983
 P 10600 1000
-F 0 "#PWR032" H 10600 850 50  0001 C CNN
+F 0 "#PWR030" H 10600 850 50  0001 C CNN
 F 1 "+3V3" H 10600 1140 50  0000 C CNN
 F 2 "" H 10600 1000 50  0001 C CNN
@@
 V_BAT
 $Comp
-L GND #PWR?
+L GND #PWR031
 U 1 1 5A13340D
 P 9950 1750
-F 0 "#PWR?" H 9950 1500 50  0001 C CNN
+F 0 "#PWR031" H 9950 1500 50  0001 C CNN
 F 1 "GND" H 9950 1600 50  0000 C CNN
 F 2 "" H 9950 1750 50  0001 C CNN
@@
 	1    0    0    -1
 $EndComp
+Text Notes 4150 2600 0    62   ~ 0
+18\n0\n1\n2\n3\n4\n5\n6/A0\n7/A1\n8/A2\n
+Text Notes 1450 2600 0    62   ~ 0
+9/A3\n10/A4\n11/A5\n12/A6\n13/A7\n14/A8\n15\n16\n17
 $EndSCHEMATC

Commit message: Added BOM
Needs update of some component footprints
Parts:
- D1, D2: symbol LED -> LED-RESCUE-ILV2-7-5_Clock
- J2: symbol USB_OTG -> USB_OTG-RESCUE-ILV2-7-5_Clock
- R13: value R -> 3.3K
Other:
- note added: "ChipKIT DP32\nPins in blue"
- note removed: "NEEDS PROG RESISTOR VALUE"
Changed lines of the file:
@@
 EESchema Schematic File Version 2
+LIBS:ILV2-7-5_Clock-rescue
 LIBS:power
 LIBS:device
@@
 LIBS:contrib
 LIBS:valves
-LIBS:OpenBCI
-LIBS:Solutions
-LIBS:Tympan
 LIBS:ILV2-7-5_Clock-cache
 EELAYER 25 0
@@
 $EndComp
 $Comp
-L USB_OTG J2
+L USB_OTG-RESCUE-ILV2-7-5_Clock J2
 U 1 1 5A04E172
 P 8150 1300
@@
 $EndComp
 $Comp
-L LED D1
+L LED-RESCUE-ILV2-7-5_Clock D1
 U 1 1 5A073B5F
 P 6000 4000
@@
 P 8150 2750
 F 0 "R13" V 8230 2750 50  0000 C CNN
-F 1 "R" V 8150 2750 50  0000 C CNN
+F 1 "3.3K" V 8150 2750 50  0000 C CNN
 F 2 "Capacitors_SMD:C_0603" V 8080 2750 50  0001 C CNN
 F 3 "" H 8150 2750 50  0001 C CNN
@@
 $EndComp
 $Comp
-L LED D2
+L LED-RESCUE-ILV2-7-5_Clock D2
 U 1 1 5A07AFE9
 P 6600 2100
@@
 	1    0    0    -1
 $EndComp
-Text Notes 7050 2200 0    60   ~ 0
-NEEDS PROG RESISTOR VALUE
 Text Label 9650 2500 0    60   ~ 0
 V_BAT
@@
 Text Notes 1450 2600 0    62   ~ 0
 9/A3\n10/A4\n11/A5\n12/A6\n13/A7\n14/A8\n15\n16\n17
+Text Notes 1750 3300 0    60   ~ 0
+ChipKIT DP32\nPins in blue
 $EndSCHEMATC

Commit message: CHANGED FROM BATTERY TO 24V SUPPLY
Parts:
- removed B1: JS_2_Battery, OpenBCI:JST_RA_SMT, symbol JS_2_Battery
- removed C12, C20: 10uF, Capacitors_SMD:C_0603, symbol C
- removed C14: 22uF 6.3V, Capacitors_SMD:C_0603, symbol C
- removed C19: 470pF 50V, Capacitors_SMD:C_0603, symbol C
- removed D2: LED, Capacitors_SMD:C_0603, symbol LED-RESCUE-ILV2-7-5_Clock
- removed L1: 10uH 1.2A, Capacitors_SMD:C_1210, symbol L
- removed R12: 1K, Capacitors_SMD:C_0603, symbol R
- removed R13: 3.3K, Capacitors_SMD:C_0603, symbol R
- removed R14: 10K, Capacitors_SMD:C_0603, symbol R
- removed R15: 150K, Capacitors_SMD:C_0603, symbol R
- removed R7, R8: 100K, Capacitors_SMD:C_0603, symbol R
- removed U4: MCP73831, TO_SOT_Packages_SMD:SOT-23-5, symbol MCP73831
- removed U6: MIC5317, TO_SOT_Packages_SMD:SOT-23-5, symbol MIC5317
- removed U7: LMR62421, TO_SOT_Packages_SMD:SOT-23-5, symbol LMR62421
- added D2: 500mA 30V, Capacitors_SMD:C_0603, symbol D
- added J3: BARREL_JACK, symbol BARREL_JACK
- added U4: TLV76033DBZR, TO_SOT_Packages_SMD:SOT-23, symbol TLV76033DBZR
- U8: value MIC5317 -> TC1014-2.5VCT713
Connections:
- net labels added: V_IN
- net labels removed: BAT_CHRG, V_BAT
- wire segments 196 -> 157
Other:
- moved on the sheet: C17, D3, J1, J2, SW3

Commit message: Updated Schematic with parts for desk clock
Parts:
- added R7, R8: 22R, Capacitors_SMD:C_0603, symbol Device:R
- BT1: symbol Battery_Cell -> Device:Battery_Cell
- C1, C10, C11, C13, C15, C16, C18, C2, C21, C3, C4, C5, C6, C7, C8, C9: symbol C -> Device:C
- C17: footprint Capacitors_SMD:C_0603 -> Capacitors_THT:CP_Radial_D5.0mm_P2.00mm; symbol C -> Device:C
- D1: symbol LED-RESCUE-ILV2-7-5_Clock -> ILV2-7-5_Clock-rescue:LED-RESCUE-ILV2-7-5_Clock
- D2, D3: symbol D -> Device:D
- J1: symbol CONN_01X05 -> ILV2-7-5_Clock-rescue:CONN_01X05
- J2: symbol USB_OTG-RESCUE-ILV2-7-5_Clock -> ILV2-7-5_Clock-rescue:USB_OTG-RESCUE-ILV2-7-5_Clock
- J3: footprint (none) -> Connectors:Barrel_Jack_CUI_PJ-102AH; symbol BARREL_JACK -> ILV2-7-5_Clock-rescue:BARREL_JACK
- Q1, Q3: symbol BSS84_PMOS_GSD -> Solutions1:BSS84_PMOS_GSD
- Q2, Q4: symbol BSS138 -> ILV2-7-5_Clock-rescue:BSS138
- R1, R10, R11, R2, R3, R4, R5, R6, R9: symbol R -> Device:R
- SW1, SW2, SW4: footprint OpenBCI:PTS810 -> Solutions:PTS810; symbol TACT_SWITCH -> OpenBCI:TACT_SWITCH
- SW3: footprint Solutions:PCM12SMTR -> Solutions:C&K_OS102011MS2QN1; symbol CJS1200 -> OpenBCI:CJS1200
- U1: symbol DS3231M -> Solutions1:DS3231M
- U2: symbol 74HC2G14 -> Solutions1:74HC2G14
- U3: symbol PIC32MX250F128B -> Solutions1:PIC32MX250F128B
- U4: symbol TLV76033DBZR -> Solutions1:TLV76033DBZR
- U5: symbol MAX6920 -> Solutions1:MAX6920
- U8: symbol MIC5317 -> Solutions1:MIC5317
- VFD1: symbol ILV2-7/5 -> ILV2-7-5_Clock-rescue:ILV2-7_5
- Y1: symbol Crystal -> Device:Crystal
Connections:
- net D+: now also R7.2; no longer J2.3 (D+)
- net D-: now also R8.2; no longer J2.2 (D-)
- net BAT_SENS: no longer names the net of U3.25 (RB14)
- new net: J2.2 (D-), R8.1
- new net: J2.3 (D+), R7.1
Other:
- moved on the sheet: D2

Commit message: re routed the board. added new footprints
Parts:
- removed R2: 680R, Capacitors_SMD:C_0603, symbol Device:R
- J3: footprint Connectors:Barrel_Jack_CUI_PJ-102AH -> Solutions:DC_PWR_PJ-006B
- SW1, SW2, SW4: footprint Solutions:PTS810 -> Solutions:D6_SPST_SW
- SW3: value PCM12SMTR -> GF-1123-1110; footprint Solutions:C&K_OS102011MS2QN1 -> Solutions:SW_GF-1123-1110; symbol OpenBCI:CJS1200 -> Switch:SW_DIP_x01
- Y1: footprint Solutions:IQD_HC49_XTAL -> Solutions:TXC_5mmX2mm
Connections:
- net +24V: now also C17.1, J3.1; no longer D3.1 (K), SW3.3 (T), U5.1 (VBB)
- net BLANK: now also U3.7 (RB2); no longer U3.24 (RB13)
- net GND: now also D3.2 (A); no longer J3.2, J3.3
- net VFD_EN: now also U3.24 (RB13); no longer U3.7 (RB2)
- net V_IN: now also U5.1 (VBB)
- net at U3.10 (OSC2/RA3): now also C4.1, Y1.2
- new net: D3.1 (K), J3.2, J3.3
Other:
- note added: "18\n0\n1\n2\n3\n4\n5\nA0/6\nA1/7\nA2/8\n"
- note removed: "18\n0\n1\n2\n3\n4\n5\n6/A0\n7/A1\n8/A2\n"
- moved on the sheet: C10, C4, C9, D1, D2, D3, J1, R10, R11, R9, SW1, SW2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

Commit message: Minor Changes
Parts:
- Q1, Q3: symbol Solutions1:BSS84_PMOS_GSD -> Transistor_FET:BSS84
- SW1, SW2, SW4: symbol OpenBCI:TACT_SWITCH -> Solutions:TACT_SWITCH
- U1: symbol Solutions1:DS3231M -> Solutions:DS3231M
- U2: symbol Solutions1:74HC2G14 -> Solutions:74HC2G14
- U3: symbol Solutions1:PIC32MX250F128B -> Solutions:PIC32MX250F128B
- U4: symbol Solutions1:TLV76033DBZR -> Solutions:TLV76033DBZR
- U5: symbol Solutions1:MAX6920 -> Solutions:MAX6920
- U8: symbol Solutions1:MIC5317 -> Solutions:MIC5317
Other:
- note added: "ADD A SPEAKER TO THIS"
Changed lines of the file:
@@
 EESchema Schematic File Version 4
-LIBS:ILV2-7-5_Clock-cache
 EELAYER 26 0
 EELAYER END
@@
 $EndComp
 $Comp
-L Solutions1:PIC32MX250F128B U3
+L Solutions:PIC32MX250F128B U3
 U 1 1 5A03A397
 P 2950 2150
@@
 $EndComp
 $Comp
-L Solutions1:DS3231M U1
+L Solutions:DS3231M U1
 U 1 1 5A03A791
 P 2250 5050
@@
 $EndComp
 $Comp
-L Solutions1:MAX6920 U5
+L Solutions:MAX6920 U5
 U 1 1 5A03AB62
 P 9050 5150
@@
 $EndComp
 $Comp
-L Solutions1:MIC5317 U8
+L Solutions:MIC5317 U8
 U 1 1 5A04E091
 P 11600 1150
@@
 $EndComp
 $Comp
-L Solutions1:74HC2G14 U2
+L Solutions:74HC2G14 U2
 U 1 1 5A0513A7
 P 2500 6650
@@
 $EndComp
 $Comp
-L Solutions1:BSS84_PMOS_GSD Q1
+L Transistor_FET:BSS84 Q1
 U 1 1 5A05E086
 P 5000 6350
@@
 $EndComp
 $Comp
-L Solutions1:BSS84_PMOS_GSD Q3
+L Transistor_FET:BSS84 Q3
 U 1 1 5A062F32
 P 6550 6350
@@
 $EndComp
 $Comp
-L OpenBCI:TACT_SWITCH SW2
+L Solutions:TACT_SWITCH SW2
 U 1 1 5A073A78
 P 5650 4050
@@
 $EndComp
 $Comp
-L OpenBCI:TACT_SWITCH SW1
+L Solutions:TACT_SWITCH SW1
 U 1 1 5A073B03
 P 5650 3150
@@
 $EndComp
 $Comp
-L OpenBCI:TACT_SWITCH SW4
+L Solutions:TACT_SWITCH SW4
 U 1 1 5A08B7A0
 P 5900 2400
@@
 ChipKIT DP32\nPins in blue
 $Comp
-L Solutions1:TLV76033DBZR U4
+L Solutions:TLV76033DBZR U4
 U 1 1 5AD4ED0F
 P 9950 1000
@@
 Wire Wire Line
 	11650 2650 11750 2650
+Text Notes 1650 3150 0    60   ~ 0
+ADD A SPEAKER TO THIS
 $EndSCHEMATC
