File: ILV2-7-5_Clock/_saved_ILV2-7-5_Clock.sch (KiCad schematic (older format))
At the start: 62 parts, among them J1 CONN_01X05, J2 USB_OTG, Q1 BSS84, Q2 BSS138, Q3 BSS84, Q4 BSS138, SW1 TACT_SWITCH, SW2 TACT_SWITCH, SW3 PCM12SMTR, SW4 TACT_SWITCH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

Commit message: Finished first draft of pub and zone fills
Parts:
- J1: footprint Pin_Headers:Pin_Header_Straight_1x05_Pitch1.00mm -> Pin_Headers:Pin_Header_Straight_1x05_Pitch2.54mm
Changed lines of the file:
@@
 F 0 "J1" H 5500 1700 50  0000 C CNN
 F 1 "CONN_01X05" V 5600 1400 50  0000 C CNN
-F 2 "Pin_Headers:Pin_Header_Straight_1x05_Pitch1.00mm" H 5500 1400 50  0001 C CNN
+F 2 "Pin_Headers:Pin_Header_Straight_1x05_Pitch2.54mm" H 5500 1400 50  0001 C CNN
 F 3 "" H 5500 1400 50  0001 C CNN
 	1    5500 1400
@@
 INT/SQW
 $Comp
-L +5V #PWR029
+L +5V #PWR028
 U 1 1 5A1216E5
 P 8500 900
-F 0 "#PWR029" H 8500 750 50  0001 C CNN
+F 0 "#PWR028" H 8500 750 50  0001 C CNN
 F 1 "+5V" H 8500 1040 50  0000 C CNN
 F 2 "" H 8500 900 50  0001 C CNN
@@
 Connection ~ 11000 1050
 $Comp
-L +5V #PWR031
+L +5V #PWR029
 U 1 1 5A122390
 P 6900 1850
-F 0 "#PWR031" H 6900 1700 50  0001 C CNN
+F 0 "#PWR029" H 6900 1700 50  0001 C CNN
 F 1 "+5V" H 6900 1990 50  0000 C CNN
 F 2 "" H 6900 1850 50  0001 C CNN
@@
 	9500 1050 9400 1050
 $Comp
-L +3V3 #PWR032
+L +3V3 #PWR030
 U 1 1 5A123983
 P 10600 1000
-F 0 "#PWR032" H 10600 850 50  0001 C CNN
+F 0 "#PWR030" H 10600 850 50  0001 C CNN
 F 1 "+3V3" H 10600 1140 50  0000 C CNN
 F 2 "" H 10600 1000 50  0001 C CNN
@@
 V_BAT
 $Comp
-L GND #PWR?
+L GND #PWR031
 U 1 1 5A13340D
 P 9950 1750
-F 0 "#PWR?" H 9950 1500 50  0001 C CNN
+F 0 "#PWR031" H 9950 1500 50  0001 C CNN
 F 1 "GND" H 9950 1600 50  0000 C CNN
 F 2 "" H 9950 1750 50  0001 C CNN

Commit message: Added mount holes, fixed the inductor footprint size
Parts:
- L1: footprint Capacitors_SMD:C_0603 -> Capacitors_SMD:C_1210
Changed lines of the file:
@@
 F 0 "L1" V 11000 2750 50  0000 C CNN
 F 1 "10uH 1.2A" V 11125 2750 50  0000 C CNN
-F 2 "Capacitors_SMD:C_0603" H 11050 2750 50  0001 C CNN
+F 2 "Capacitors_SMD:C_1210" H 11050 2750 50  0001 C CNN
 F 3 "" H 11050 2750 50  0001 C CNN
 	1    11050 2750
